File: freezer.kicad_pcb (KiCad board)
At the start: 2 copper layers, 50 x 200 mm, 77 parts, among them J1 audio in, J10 audio_out, J11 audio out, J2 audio_in, J3 Eurorack power, J4 trigger in, J5 trigger_in, J6 CV1 in, J7 CV2 in, J8 cv2_in, J9 cv1_in, Q1 2N3904, SW1 SW_SPDT, SW2 SW_SPDT, SW3 button, SW4 Bypass, U1 TL072, U2 23LCV1024-I_P, U3 23LCV1024-I_P, U4 LM4040 5V, U5 MCP6004, U6 MCP3201_CI_P, U7 L7805, U8 MCP4921

Commit message: more work
Parts:
- added D3: 1N4148, Diode_THT:D_DO-35_SOD27_P7.62mm_Horizontal, F.Cu at (77.2, 168.2)
- C10: footprint Capacitor_THT:CP_Radial_D5.0mm_P2.00mm -> Capacitor_THT:CP_Radial_D6.3mm_P2.50mm
- D1: footprint Connector_Molex:Molex_KK-254_AE-6410-02A_1x02_P2.54mm_Vertical -> LED_THT:LED_D5.0mm
- R1, R10, R11, R12, R13, R14, R15, R16, R17, R18, R19, R2, R20, R21, R22, R23, R24, R25, R26, R27, R28, R29, R3, R4, R5, R6, R7, R8, R9: footprint R_silkvalue:R_Axial_DIN0207_L6.3mm_D2.5mm_P2.54mm_Vertical_silkvalue -> R_silkvalue:R_Axial_DIN0207_L6.3mm_D2.5mm_P7.62mm_Horizontal_silkvalue
- U6: value MCP3201_CI_P -> MCP3201
- moved J4 156.0 mm to (87.5, 198.0)
- moved J5 128.8 mm to (73.5, 182.0)
- moved R12 122.7 mm to (71.8, 177.2)
- moved Q1 111.7 mm to (76.0, 173.2)
- moved R13 103.6 mm to (73.0, 162.0), turned to 270 degrees
- moved H1 100.1 mm to (109.2, 59.8)
- moved R28 97.0 mm to (108.8, 145.5), turned to 180 degrees
- moved R14 95.9 mm to (80.5, 159.0), turned to 270 degrees
- moved R11 79.6 mm to (123.5, 155.2), turned to 270 degrees
- moved U5 75.2 mm to (111.8, 153.5), turned to 0 degrees
- moved C12 67.6 mm to (108.5, 158.5), turned to 270 degrees
- moved C13 63.1 mm to (120.8, 145.8)
- moved R9 58.4 mm to (123.2, 180.5)
- moved R21 57.8 mm to (108.8, 134.5)
- moved R26 55.3 mm to (111.8, 141.2)
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Other:
- board size 50 x 200 mm -> 75 x 104.5 mm

Commit message: before moving the DAC ADC chips
Parts:
- U2, U3: value 23LCV1024-I_P -> 23LCV1024
- moved R1 30.6 mm to (74.4, 142.2), turned to 90 degrees
- moved R2 15.4 mm to (51.6, 135.4)
- moved D2 14.9 mm to (53.6, 87.4)
- moved R27 14.6 mm to (51.6, 121.7)
- moved R14 13.3 mm to (72.9, 169.9), turned to 0 degrees
- moved R7 11.1 mm to (94.2, 146.6), turned to 270 degrees
- moved R13 10.9 mm to (83.1, 166.1), turned to 180 degrees
- moved R12 10.8 mm to (80.0, 184.2), turned to 90 degrees
- moved D3 8.17 mm to (83.1, 174.0), turned to 270 degrees
- moved C9 7.56 mm to (74.4, 146.1), turned to 270 degrees
- moved C15 7.53 mm to (114.0, 132.3)
- moved SW3 5.05 mm to (53.3, 97.3)
- moved C18 4.29 mm to (86.4, 170.2)
- moved C7 4.19 mm to (77.7, 155.4)
- moved C10 4.01 mm to (79.0, 132.8)
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Connections:
- A1 pad 7: CS_0 -> CS_1
- A1 pad 8: CS_1 -> CS_0
- RV1 pad 1: GND -> +5V
- RV1 pad 3: +5V -> GND
- RV2 pad 1: GND -> +5V
- RV2 pad 3: +5V -> GND
Routing:
- net SCK: track 0.00 -> 130.2 mm
- net COPI: track 0.00 -> 107.2 mm
- net CS_1: track 0.00 -> 86.6 mm
- net CS_0: track 0.00 -> 77.3 mm
- net CIPO: track 0.00 -> 69.2 mm
- net +12V: track 0.00 -> 55.4 mm
- net -12V: track 0.00 -> 54.9 mm
- net Net-(A1-Pad14): track 0.00 -> 51.8 mm
- net +5V: track 0.00 -> 50.1 mm
- net SWITCH_2: track 0.00 -> 47.5 mm
- net Net-(C15-Pad2): track 0.00 -> 46.0 mm
- net Net-(C14-Pad2): track 0.00 -> 45.5 mm
- net Net-(R8-Pad2): track 0.00 -> 39.0 mm
- net BUTTON: track 0.00 -> 38.3 mm
- net CV1_IN: track 0.00 -> 35.7 mm
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Other:
- board text added: "GND"
- board text added: "LED GND is swapped!"

Commit message: routing done!
Parts:
- removed H1: MountingHole_Pad, MountingHole:MountingHole_3.2mm_M3
- moved R24 46.6 mm to (119.6, 184.9), turned to 90 degrees
- moved C15 40.5 mm to (99.1, 169.9), turned to 0 degrees
- moved C11 36.9 mm to (112.5, 136.1)
- moved U8 36.8 mm to (112.5, 139.2)
- moved R23 35.3 mm to (123.2, 174.8), turned to 270 degrees
- moved R21 33.6 mm to (97.5, 167.4), turned to 90 degrees
- moved C14 32.4 mm to (94.0, 164.9), turned to 270 degrees
- moved R25 27.0 mm to (123.4, 131.3), turned to 270 degrees
- moved R22 23.7 mm to (101.6, 157.2), turned to 270 degrees
- moved U6 22.0 mm to (101.1, 139.2)
- moved C8 20.8 mm to (102.4, 134.9), turned to 90 degrees
- moved C17 15.5 mm to (116.3, 178.6), turned to 90 degrees
- moved R11 15.0 mm to (119.1, 169.7), turned to 90 degrees
- moved R28 12.0 mm to (97.8, 143.0), turned to 90 degrees
- moved R26 11.5 mm to (123.4, 144.0), turned to 270 degrees
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Connections:
- U5 pad 10: Net-(C13-Pad1) -> Net-(R23-Pad1)
- U5 pad 12: Net-(U5-Pad12) -> Net-(R11-Pad1)
- U5 pad 13: Net-(R23-Pad1) -> Net-(C13-Pad1)
- U5 pad 14: Net-(R23-Pad1) -> Net-(R11-Pad2)
- U5 pad 8: Net-(R11-Pad2) -> Net-(R23-Pad1)
- U5 pad 9: Net-(R11-Pad1) -> Net-(U5-Pad9)
- U8 pad 8: Net-(U5-Pad12) -> Net-(U5-Pad9)
Routing:
- net +5V: track 50.1 -> 240.7 mm, vias 0 -> 1
- net CV_CH_2: track 0.00 -> 65.7 mm
- net CV_CH_1: track 0.00 -> 65.1 mm
- net Net-(R5-Pad2): track 0.00 -> 62.4 mm
- net -12V: track 54.9 -> 114.7 mm
- net Net-(R11-Pad2): track 0.00 -> 51.7 mm
- net IN_TRIGGER: track 0.00 -> 50.7 mm
- net Net-(C14-Pad2): track 45.5 -> 94.8 mm
- net Net-(C15-Pad2): track 46.0 -> 95.4 mm
- net Net-(C18-Pad1): track 0.00 -> 40.1 mm
- net REF_-5V: track 0.00 -> 35.6 mm
- net Net-(U5-Pad9): track 0.00 -> 35.3 mm
- net COPI: track 107.2 -> 76.0 mm, vias 0 -> 2
- net Net-(A1-Pad14): track 51.8 -> 20.9 mm
- net Net-(R18-Pad1): track 0.00 -> 29.8 mm, vias 0 -> 1
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- added copper zone on B.Cu, net GND
Other:
- board size 75 x 104.5 mm -> 75 x 102 mm
- board text added: "lay down CPs"
