File: midi2trigger.kicad_pcb (KiCad board)
At the start: 2 copper layers, 74 x 175 mm, 75 parts, among them J1 MIDI IN, J10 GATE7, J11 GATE8, J12 GATE9, J13 GATE10, J14 GATE11, J15 GATE12, J2 Eurorack power, J3 GATE1, J4 GATE2, J5 GATE3, J6 GATE4, J7 MIDI OUT, J8 GATE5, J9 GATE6, U1 TL074, U2 6N137, U3 L7805, U4 TL074, U5 TL074

Commit message: as sent to jlcpcb
Connections:
- A1 pad 1: (no net) -> MIDI_OUT
- R14 pad 1: MIDI_IN -> MIDI_OUT
Routing:
- net Net-(J13-PadT): track 0.00 -> 11.1 mm
- net MIDI_OUT: track 0.00 -> 3.78 mm
- net MIDI_IN: track 21.8 -> 21.0 mm
Changed lines of the file:
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@@
     (thickness 1.6)
     (drawings 26)
-    (tracks 398)
+    (tracks 402)
     (zones 0)
     (modules 75)
-    (nets 61)
+    (nets 62)
   )
   (page A4 portrait)
@@
   (net 59 "Net-(R6-Pad1)")
   (net 60 "Net-(R8-Pad1)")
+  (net 61 MIDI_OUT)
   (net_class Default "This is the default net class."
     (clearance 0.2)
@@
     (add_net GND)
     (add_net MIDI_IN)
+    (add_net MIDI_OUT)
     (add_net "Net-(D1-Pad1)")
     (add_net "Net-(D1-Pad2)")
@@
       (effects (font (size 1 1) (thickness 0.15)))
     )
-    (fp_text user %R (at 3.81 3.81 90) (layer F.Fab)
-      (effects (font (size 1 1) (thickness 0.15)))
-    )
-    (fp_arc (start 3.81 -1.33) (end 2.81 -1.33) (angle -180) (layer F.SilkS) (width 0.12))
     (fp_line (start 1.635 -1.27) (end 6.985 -1.27) (layer F.Fab) (width 0.1))
     (fp_line (start 6.985 -1.27) (end 6.985 8.89) (layer F.Fab) (width 0.1))
@@
     (fp_line (start 8.7 9.15) (end 8.7 -1.55) (layer F.CrtYd) (width 0.05))
     (fp_line (start 8.7 -1.55) (end -1.1 -1.55) (layer F.CrtYd) (width 0.05))
+    (fp_text user %R (at 3.81 3.81 90) (layer F.Fab)
+      (effects (font (size 1 1) (thickness 0.15)))
+    )
+    (fp_arc (start 3.81 -1.33) (end 2.81 -1.33) (angle -180) (layer F.SilkS) (width 0.12))
     (pad 8 thru_hole oval (at 7.62 0 270) (size 1.6 1.6) (drill 0.8) (layers *.Cu *.Mask)
       (net 4 +5V))
@@
       (net 56 "Net-(J7-Pad3)"))
     (pad 1 thru_hole circle (at 0 0 90) (size 1.6 1.6) (drill 0.8) (layers *.Cu *.Mask)
-      (net 39 MIDI_IN))
+      (net 61 MIDI_OUT))
     (model ${KISYS3DMOD}/Resistor_THT.3dshapes/R_Axial_DIN0207_L6.3mm_D2.5mm_P10.16mm_Horizontal.wrl
       (at (xyz 0 0 0))
@@
       (effects (font (size 1 1) (thickness 0.15)))
     )
-    (fp_text user K (at 0 1.905 90) (layer F.SilkS)
-      (effects (font (size 1 1) (thickness 0.15)))
-    )
-    (fp_text user %R (at 5.23 0 90) (layer F.Fab)
-      (effects (font (size 0.8 0.8) (thickness 0.12)))
-    )
     (fp_line (start 3.08 -1) (end 3.08 1) (layer F.Fab) (width 0.1))
     (fp_line (start 3.08 1) (end 7.08 1) (layer F.Fab) (width 0.1))
@@
     (fp_line (start 11.21 1.25) (end 11.21 -1.25) (layer F.CrtYd) (width 0.05))
     (fp_line (start 11.21 -1.25) (end -1.05 -1.25) (layer F.CrtYd) (width 0.05))
+    (fp_text user K (at 0 1.905 90) (layer F.SilkS)
+      (effects (font (size 1 1) (thickness 0.15)))
+    )
+    (fp_text user %R (at 5.23 0 90) (layer F.Fab)
+      (effects (font (size 0.8 0.8) (thickness 0.12)))
+    )
     (pad 2 thru_hole oval (at 10.16 0 90) (size 1.6 1.6) (drill 0.8) (layers *.Cu *.Mask)
       (net 6 "Net-(D1-Pad2)"))
@@
       (effects (font (size 1 1) (thickness 0.15)))
     )
-    (fp_text user %R (at 3.81 7.62 90) (layer F.Fab)
-      (effects (font (size 1 1) (thickness 0.15)))
-    )
-    (fp_arc (start 3.81 -1.33) (end 2.81 -1.33) (angle -180) (layer F.SilkS) (width 0.12))
     (fp_line (start 1.635 -1.27) (end 6.985 -1.27) (layer F.Fab) (width 0.1))
     (fp_line (start 6.985 -1.27) (end 6.985 16.51) (layer F.Fab) (width 0.1))
@@
     (fp_line (start 9.15 16.85) (end 9.15 -1.6) (layer F.CrtYd) (width 0.05))
     (fp_line (start 9.15 -1.6) (end -1.55 -1.6) (layer F.CrtYd) (width 0.05))
+    (fp_text user %R (at 3.81 7.62 90) (layer F.Fab)
+      (effects (font (size 1 1) (thickness 0.15)))
+    )
+    (fp_arc (start 3.81 -1.33) (end 2.81 -1.33) (angle -180) (layer F.SilkS) (width 0.12))
     (pad 14 thru_hole oval (at 7.62 0 270) (size 2.4 1.6) (drill 0.8) (layers *.Cu *.Mask)
       (net 54 "Net-(R29-Pad1)"))
@@
       (effects (font (size 1 1) (thickness 0.15)))
     )
-    (fp_text user %R (at 1.25 0 90) (layer F.Fab)
-      (effects (font (size 0.68 0.68) (thickness 0.102)))
-    )
     (fp_line (start -0.45 -1.05) (end -0.45 1.05) (layer F.Fab) (width 0.1))
     (fp_line (start -0.45 1.05) (end 2.95 1.05) (layer F.Fab) (width 0.1))
@@
     (fp_line (start 3.55 1.3) (end 3.55 -1.3) (layer F.CrtYd) (width 0.05))
     (fp_line (start 3.55 -1.3) (end -1.05 -1.3) (layer F.CrtYd) (width 0.05))
+    (fp_text user %R (at 1.25 0 90) (layer F.Fab)
+      (effects (font (size 0.68 0.68) (thickness 0.102)))
+    )
     (pad 2 thru_hole circle (at 2.5 0 270) (size 1.6 1.6) (drill 0.8) (layers *.Cu *.Mask)
       (net 1 +12V))
@@
       (effects (font (size 1 1) (thickness 0.15)))
     )
-    (fp_text user %R (at 1.25 0 90) (layer F.Fab)
-      (effects (font (size 0.68 0.68) (thickness 0.102)))
-    )
     (fp_line (start -0.45 -1.05) (end -0.45 1.05) (layer F.Fab) (width 0.1))
     (fp_line (start -0.45 1.05) (end 2.95 1.05) (layer F.Fab) (width 0.1))
@@
     (fp_line (start 3.55 1.3) (end 3.55 -1.3) (layer F.CrtYd) (width 0.05))
     (fp_line (start 3.55 -1.3) (end -1.05 -1.3) (layer F.CrtYd) (width 0.05))
+    (fp_text user %R (at 1.25 0 90) (layer F.Fab)
+      (effects (font (size 0.68 0.68) (thickness 0.102)))
+    )
     (pad 2 thru_hole circle (at 2.5 0 90) (size 1.6 1.6) (drill 0.8) (layers *.Cu *.Mask)
       (net 3 -12V))
@@
       (effects (font (size 1 1) (thickness 0.15)))
     )
-    (fp_text user %R (at 1.25 0 90) (layer F.Fab)
-      (effects (font (size 0.68 0.68) (thickness 0.102)))
-    )
     (fp_line (start -0.45 -1.05) (end -0.45 1.05) (layer F.Fab) (width 0.1))
     (fp_line (start -0.45 1.05) (end 2.95 1.05) (layer F.Fab) (width 0.1))
@@
     (fp_line (start 3.55 1.3) (end 3.55 -1.3) (layer F.CrtYd) (width 0.05))
     (fp_line (start 3.55 -1.3) (end -1.05 -1.3) (layer F.CrtYd) (width 0.05))
+    (fp_text user %R (at 1.25 0 90) (layer F.Fab)
+      (effects (font (size 0.68 0.68) (thickness 0.102)))
+    )
     (pad 2 thru_hole circle (at 2.5 0 270) (size 1.6 1.6) (drill 0.8) (layers *.Cu *.Mask)
       (net 1 +12V))
@@
       (effects (font (size 1 1) (thickness 0.15)))
     )
-    (fp_text user %R (at 1.25 0 90) (layer F.Fab)
-      (effects (font (size 0.68 0.68) (thickness 0.102)))
-    )
     (fp_line (start -0.45 -1.05) (end -0.45 1.05) (layer F.Fab) (width 0.1))
     (fp_line (start -0.45 1.05) (end 2.95 1.05) (layer F.Fab) (width 0.1))
@@
     (fp_line (start 3.55 1.3) (end 3.55 -1.3) (layer F.CrtYd) (width 0.05))
     (fp_line (start 3.55 -1.3) (end -1.05 -1.3) (layer F.CrtYd) (width 0.05))
+    (fp_text user %R (at 1.25 0 90) (layer F.Fab)
+      (effects (font (size 0.68 0.68) (thickness 0.102)))
+    )
     (pad 2 thru_hole circle (at 2.5 0 90) (size 1.6 1.6) (drill 0.8) (layers *.Cu *.Mask)
       (net 3 -12V))
@@
       (net 39 MIDI_IN))
     (pad 17 thru_hole oval (at 15.24 -33.02 270) (size 1.6 1.6) (drill 1) (layers *.Cu *.Mask))
-    (pad 1 thru_hole rect (at 0 0 270) (size 1.6 1.6) (drill 1) (layers *.Cu *.Mask))
+    (pad 1 thru_hole rect (at 0 0 270) (size 1.6 1.6) (drill 1) (layers *.Cu *.Mask)
+      (net 61 MIDI_OUT))
     (model ${KISYS3DMOD}/Module.3dshapes/Arduino_Nano_WithMountingHoles.wrl
       (at (xyz 0 0 0))
@@
   (segment (start 113.665 150.495) (end 111.76 148.59) (width 0.4) (layer B.Cu) (net 30))
   (segment (start 116.84 150.495) (end 113.665 150.495) (width 0.4) (layer B.Cu) (net 30))
+  (segment (start 57.785 139.685) (end 57.6 139.5) (width 0.4) (layer B.Cu) (net 31))
+  (segment (start 57.785 150.495) (end 57.785 139.685) (width 0.4) (layer B.Cu) (net 31))
   (segment (start 53.34 165.1) (end 53.34 163.83) (width 0.4) (layer B.Cu) (net 32))
   (segment (start 53.67 163.5) (end 57.6 163.5) (width 0.4) (layer B.Cu) (net 32))
@@
   (segment (start 84.54 184.87) (end 84.455 184.785) (width 0.4) (layer B.Cu) (net 39))
   (segment (start 84.54 188) (end 84.54 184.87) (width 0.4) (layer B.Cu) (net 39))
-  (segment (start 84.455 184.785) (end 80.645 184.785) (width 0.4) (layer B.Cu) (net 39))
-  (segment (start 70.485 186.69) (end 70.485 190.5) (width 0.4) (layer F.Cu) (net 39))
-  (segment (start 72.39 184.785) (end 70.485 186.69) (width 0.4) (layer F.Cu) (net 39))
-  (segment (start 80.645 184.785) (end 72.39 184.785) (width 0.4) (layer F.Cu) (net 39))
+  (segment (start 83.04 186.2) (end 84.455 184.785) (width 0.4) (layer F.Cu) (net 39))
+  (segment (start 72.4 186.2) (end 83.04 186.2) (width 0.4) (layer F.Cu) (net 39))
+  (segment (start 70.485 188.115) (end 72.4 186.2) (width 0.4) (layer F.Cu) (net 39))
+  (segment (start 70.485 190.5) (end 70.485 188.115) (width 0.4) (layer F.Cu) (net 39))
   (segment (start 101.640034 60.151491) (end 101.640034 178.394966) (width 0.4) (layer F.Cu) (net 40))
   (segment (start 96.133532 54.644989) (end 101.640034 60.151491) (width 0.4) (layer F.Cu) (net 40))
@@
   (segment (start 82.3 63.885) (end 82.3 63.115) (width 0.4) (layer B.Cu) (net 60))
   (segment (start 83.185 64.77) (end 82.3 63.885) (width 0.4) (layer B.Cu) (net 60))
+  (segment (start 82 186.14) (end 80.645 184.785) (width 0.4) (layer B.Cu) (net 61))
+  (segment (start 82 188) (end 82 186.14) (width 0.4) (layer B.Cu) (net 61))
   (zone (net 2) (net_name GND) (layer F.Cu) (hatch edge 0.508)
     (connect_pads (clearance 0.508))
