File: panel/midi2trigger.kicad_pcb (KiCad board)
At the start: 2 copper layers, 75 x 200 mm, 46 parts

Commit message: as sent to jlcpcb
Parts:
- removed the G*** at (78.0, 156.0)
- removed the G*** at (78.0, 132.0)
- removed the G*** at (78.0, 108.0)
- removed the G*** at (78.0, 84.0)
- removed the G*** at (78.0, 60.0)
- removed the G*** at (78.0, 36.0)
- removed the G*** at (87.0, 214.0)
- removed the G*** at (97.0, 156.0)
- removed the G*** at (97.0, 132.0)
- removed the G*** at (97.0, 108.0)
- removed the G*** at (97.0, 84.0)
- removed the G*** at (97.0, 60.0)
- removed the G*** at (97.0, 36.0)
- removed the REF** at (53.0, 23.0)
- removed the REF** at (122.0, 23.0)
- removed the REF** at (122.0, 217.0)
- removed the REF** at (53.0, 217.0)
- added G***: LOGO, midi2trigger_panel:12, F.Cu at (97.0, 156.0)
- added G***: LOGO, midi2trigger_panel:3, F.Cu at (78.0, 84.0)
- added G***: LOGO, midi2trigger_panel:2, F.Cu at (78.2, 60.0)
- added G***: LOGO, midi2trigger_panel:logo_3, F.Cu at (84.1, 213.7)
- added G***: LOGO, midi2trigger_panel:1, F.Cu at (77.6, 35.5)
- added G***: LOGO, midi2trigger_panel:11, F.Cu at (97.0, 132.0)
- added G***: LOGO, midi2trigger_panel:10, F.Cu at (97.0, 108.0)
- added G***: LOGO, midi2trigger_panel:9, F.Cu at (97.0, 84.0)
- added G***: LOGO, midi2trigger_panel:8, F.Cu at (97.0, 60.0)
- added G***: LOGO, midi2trigger_panel:7, F.Cu at (97.0, 36.0)
- added G***: LOGO, midi2trigger_panel:6, F.Cu at (78.0, 156.0)
- added G***: LOGO, midi2trigger_panel:5, F.Cu at (78.0, 132.0)
- added G***: LOGO, midi2trigger_panel:4, F.Cu at (78.0, 108.0)
- added REF**: Kosmo_Panel_Dual_Slotted_Mounting_Hole, Kosmo_panel_analogoutput:Kosmo_Panel_Dual_Slotted_Mounting_Hole, F.Cu at (119.0, 217.0)
- added REF**: Kosmo_Panel_Dual_Slotted_Mounting_Hole, Kosmo_panel_analogoutput:Kosmo_Panel_Dual_Slotted_Mounting_Hole, F.Cu at (53.0, 217.0)
- moved G*** 2.04 mm to (88.4, 27.0)
- moved G*** 0.92 mm to (104.8, 177.9)
- moved G*** 0.72 mm to (70.4, 177.6)
